Commit message: sim2sim

File: source/robot_lab/data/Robots/cyborg/biped_temp_1_0/urdf/biped_temp_1_0.urdf (robot description, URDF)
Before this commit: robot biped_temp_1_0, 31 links, 30 joints
Links:
- link ankle_l_pitch_link: geometry collision cylinder length=0.06 radius=0.01; visual mesh filename=../meshes/ankle_l_pitch_link.STL
- link ankle_l_roll_link: geometry collision mesh filename=../meshes/ankle_l_roll_link.STL; visual mesh filename=../meshes/ankle_l_roll_link.STL
- link ankle_r_pitch_link: geometry collision cylinder length=0.06 radius=0.01; visual mesh filename=../meshes/ankle_r_pitch_link.STL
- link ankle_r_roll_link: geometry collision mesh filename=../meshes/ankle_r_roll_link.STL; visual mesh filename=../meshes/ankle_r_roll_link.STL
- link arm_l_01_link: geometry collision cylinder length=0.1 radius=0.054; visual mesh filename=../meshes/arm_l_01_link.STL
- link arm_l_02_link: geometry collision cylinder length=0.055 radius=0.045; visual mesh filename=../meshes/arm_l_02_link.STL
- link arm_l_03_link: geometry collision cylinder length=0.09 radius=0.045; visual mesh filename=../meshes/arm_l_03_link.STL
- link arm_l_04_link: geometry collision cylinder length=0.14 radius=0.04; visual mesh filename=../meshes/arm_l_04_link.STL
- link arm_l_05_link: geometry collision cylinder length=0.08 radius=0.04; visual mesh filename=../meshes/arm_l_05_link.STL
- link arm_l_06_link: geometry collision cylinder length=0.052 radius=0.036; visual mesh filename=../meshes/arm_l_06_link.STL
- link arm_l_07_link: geometry collision cylinder length=0.015 radius=0.04; visual mesh filename=../meshes/arm_l_07_link.STL
- link arm_r_01_link: geometry collision cylinder length=0.1 radius=0.054; visual mesh filename=../meshes/arm_r_01_link.STL
- link arm_r_02_link: geometry collision cylinder length=0.055 radius=0.045; visual mesh filename=../meshes/arm_r_02_link.STL
- link arm_r_03_link: geometry collision cylinder length=0.09 radius=0.045; visual mesh filename=../meshes/arm_r_03_link.STL
- link arm_r_04_link: geometry collision cylinder length=0.14 radius=0.04; visual mesh filename=../meshes/arm_r_04_link.STL
- link arm_r_05_link: geometry collision cylinder length=0.08 radius=0.04; visual mesh filename=../meshes/arm_r_05_link.STL
- link arm_r_06_link: geometry collision cylinder length=0.052 radius=0.036; visual mesh filename=../meshes/arm_r_06_link.STL
- link arm_r_07_link: geometry collision cylinder length=0.015 radius=0.04; visual mesh filename=../meshes/arm_r_07_link.STL
- link base_link: geometry collision cylinder length=0.065 radius=0.05; collision cylinder length=0.08 radius=0.06
- link head_pitch_link: geometry collision box size=0.12 0.12 0.08; visual mesh filename=../meshes/head_pitch_link.STL
- link head_yaw_link: geometry collision cylinder length=0.08 radius=0.025; visual mesh filename=../meshes/head_yaw_link.STL
- link hip_l_pitch_link: geometry collision cylinder length=0.26 radius=0.055; visual mesh filename=../meshes/hip_l_pitch_link.STL
- link hip_l_roll_link: geometry collision cylinder length=0.065 radius=0.062; visual mesh filename=../meshes/hip_l_roll_link.STL
- link hip_l_yaw_link: geometry collision cylinder length=0.12 radius=0.064; visual mesh filename=../meshes/hip_l_yaw_link.STL
- link hip_r_pitch_link: geometry collision cylinder length=0.26 radius=0.055; visual mesh filename=../meshes/hip_r_pitch_link.STL
- link hip_r_roll_link: geometry collision cylinder length=0.065 radius=0.062; visual mesh filename=../meshes/hip_r_roll_link.STL
- link hip_r_yaw_link: geometry collision cylinder length=0.12 radius=0.064; visual mesh filename=../meshes/hip_r_yaw_link.STL
- link knee_l_pitch_link: geometry collision cylinder length=0.23 radius=0.05; visual mesh filename=../meshes/knee_l_pitch_link.STL
- link knee_r_pitch_link: geometry collision cylinder length=0.23 radius=0.05; visual mesh filename=../meshes/knee_r_pitch_link.STL
- link waist_pitch_link: geometry collision box size=0.285 0.32 0.42; visual mesh filename=../meshes/waist_pitch_link.STL
- link waist_yaw_link: geometry collision cylinder length=0.11 radius=0.052; visual mesh filename=../meshes/waist_yaw_link.STL
